File: keybraod.sch (KiCad schematic (older format))
At the start: 21 parts

Commit message: part2 complete
Yes.. part2 complete, 2 more
Parts:
- removed USB?: HRO-TYPE-C-31-M-12, symbol Type-C:HRO-TYPE-C-31-M-12
- added USB2: HRO-TYPE-C-31-M-12, Type-C:HRO-TYPE-C-31-M-12-HandSoldering, symbol Type-C:HRO-TYPE-C-31-M-12
- C1, C2, C3, C4, C5, C6, C7, C8: renamed from C?; footprint (none) -> Capacitor_SMD:C_0805_2012Metric_Pad1.15x1.40mm_HandSolder
- F1: renamed from F?; footprint (none) -> Fuse:Fuse_1206_3216Metric_Pad1.42x1.75mm_HandSolder
- J1: renamed from J?; footprint (none) -> random-keyboard-parts:Reset_Pretty-Mask
- R1, R2, R3, R4, R5, R6: renamed from R?; footprint (none) -> Resistor_SMD:R_0805_2012Metric_Pad1.15x1.40mm_HandSolder
- Resetpushbutton1: renamed from SW?; footprint (none) -> Button_Switch_SMD:SW_SPST_SKQG_WithStem
- U2: renamed from U?; footprint (none) -> random-keyboard-parts:SOT143B
- X1: renamed from X?; footprint (none) -> Crystal:Crystal_SMD_3225-4Pin_3.2x2.5mm_HandSoldering
- gave numbers to parts that had none: 1
Connections:
- net labels added: col0, col1, col10, col11, col12, col13, col14, col2, col3, col4, col5, col6, col7, col8, col9, row0, row1, row2, row3, row4
- wire segments 88 -> 91
- no-connect marks 5 -> 7
