File: keybraod.kicad_pcb (KiCad board)
At the start: 2 copper layers, 304.8 x 99.9 mm, 155 parts, among them J1 AVR-ISP-6, SW1 GRV, SW10 #9, SW11 #0, SW12 -, SW13 =, SW14 bs, SW15 pgup, SW16 tab, SW17 q, SW18 w, SW19 e, SW2 #1, SW20 r, SW21 t, SW22 y, SW23 u, SW24 i, SW25 o, SW26 p, SW27 [, SW28 ], SW29 \, SW3 #2, SW30 pgdn, SW31 caplock, SW32 a, SW33 s, SW34 d, SW35 f, SW36 g, SW37 h, SW38 j, SW39 k, SW4 #3, SW40 l, SW41 ;, SW42 ', SW43 enter, SW44 ins, SW45 lshift, SW46 z, SW47 x, SW48 c, SW49 v, SW5 #4, SW50 b, SW51 n, SW52 m, SW53 ,, SW54 ., SW55 /, SW56 rshift, SW57 up, SW58 del, SW59 ctrl, SW6 #5, SW60 lalt, SW61 cmd, SW62 spacebar, SW63 ralt, SW64 0, SW65 left, SW66 down, SW67 right, SW7 #6, SW8 #7, SW9 #8, U1 ATmega32U4-AU, U2 PRTR5V0U2X, X1 XTAL

Commit message: part3 complete
-switch pcb mirror
Parts:
- removed the R1 at (149.5, 134.2)
- added FB1: 60@100MHz, Inductor_SMD:L_0805_2012Metric_Pad1.15x1.40mm_HandSolder, B.Cu at (153.9, 44.2)
- added R2: 10k, Resistor_SMD:R_0805_2012Metric_Pad1.15x1.40mm_HandSolder, B.Cu at (149.4, 133.7)
- moved J1 63.6 mm to (183.2, 122.1)
- moved C6 30.1 mm to (143.6, 118.6), turned to 270 degrees
- moved C3 19.0 mm to (159.3, 115.1), turned to 180 degrees
- moved C5 16.4 mm to (162.4, 133.6), turned to 0 degrees
- moved R1 11.1 mm to (178.2, 130.9), turned to 180 degrees
- moved C1 3.27 mm to (173.3, 126.2)
- moved C2 3.19 mm to (173.3, 123.8)
- moved C4 2.54 mm to (147.4, 119.9)
- moved C8 2.51 mm to (167.5, 120.0)
- moved Resetpushbutton1 2.02 mm to (184.7, 129.1), turned to 0 degrees
- moved C7 0.49 mm to (147.3, 130.0)
- turned U2 to 180 degrees
- turned X1 to 90 degrees
- renumbered C2 to C1, C3 to C2, C1 to C3, R2 to R1, USB2 to USB1
Connections:
- net Net-(R3-Pad1) renamed DN
- net Net-(R4-Pad2) renamed DP
- Resetpushbutton1 pad 1: (no net) -> Net-(Resetpushbutton1-Pad1)
- Resetpushbutton1 pad 2: (no net) -> GND
- SW15 pad 2: col0 -> col14
- SW30 pad 2: col0 -> col14
- SW44 pad 2: col0 -> col14
- SW58 pad 2: col0 -> col14
- SW67 pad 2: col0 -> col14
- U1 pad 12: Net-(U1-Pad12) -> (no net)
- U1 pad 18: Net-(U1-Pad18) -> (no net)
- U1 pad 27: col0 -> col14
- U1 pad 42: Net-(U1-Pad42) -> (no net)
- USB1 pad 3: Net-(USB2-Pad3) -> (no net)
- USB1 pad 9: Net-(USB2-Pad9) -> (no net)
Routing:
- net col0: track 0.00 -> 4372.4 mm, vias 0 -> 29
- net GND: track 0.00 -> 309.5 mm, vias 0 -> 105
- net col14: track 0.00 -> 223.3 mm, vias 0 -> 1
- net +5V: track 0.00 -> 194.4 mm, vias 0 -> 9
- net DP: track 0.00 -> 80.1 mm
- net DN: track 0.00 -> 77.0 mm
- net RESET: track 0.00 -> 43.2 mm, vias 0 -> 2
- net MOSI: track 0.00 -> 32.5 mm
- net MISO: track 0.00 -> 29.2 mm
- net SCK: track 0.00 -> 28.6 mm
- net VCC: track 0.00 -> 23.3 mm, vias 0 -> 2
- net XTAL1: track 0.00 -> 12.8 mm
- net XTAL2: track 0.00 -> 12.0 mm
- net Net-(D8-Pad2): track 0.00 -> 10.3 mm
- net Net-(D14-Pad2): track 0.00 -> 6.79 mm
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- added copper zone on B.Cu, net GND
- added copper zone on F.Cu, net GND
