File: matrix.sch (KiCad schematic (older format))
At the start: 134 parts, among them SW1 GRV, SW10 #9, SW11 #0, SW12 -, SW13 =, SW14 bs, SW15 pgup, SW16 tab, SW17 q, SW18 w, SW19 e, SW2 #1, SW20 r, SW21 t, SW22 y, SW23 u, SW24 i, SW25 o, SW26 p, SW27 [, SW28 ], SW29 \\, SW3 #2, SW30 pgdn, SW31 caplock, SW32 a, SW33 s, SW34 d, SW35 f, SW36 g, SW37 h, SW38 j, SW39 k, SW4 #3, SW40 l, SW41 ;, SW42 ', SW43 enter, SW44 ins, SW45 lshift, SW46 z, SW47 x, SW48 c, SW49 v, SW5 #4, SW50 b, SW51 n, SW52 m, SW53 ,, SW54 ., SW55 /, SW56 rshift, SW57 up, SW58 del, SW59 ctrl, SW6 #5, SW60 lalt, SW61 cmd, SW62 spacebar, SW63 ralt, SW64 0, SW65 left, SW66 down, SW67 right, SW7 #6, SW8 #7, SW9 #8

Commit message: part3 complete
-switch pcb mirror
Connections:
- net col0: no longer SW15.2, SW30.2, SW44.2, SW58.2, SW67.2
- new net col14: SW15.2, SW30.2, SW44.2, SW58.2, SW67.2
Changed lines of the file:
@@
 $EndComp
-Wire Wire Line
-	9100 1800 9500 1800
 Wire Wire Line
 	9500 1200 9500 1500
 Connection ~ 9500 1500
-Wire Wire Line
-	9500 1500 9500 1800
-Connection ~ 9500 1800
-Text GLabel 1250 1800 0    50   Input ~ 0
-row0
 Wire Wire Line
 	1250 1800 1400 1800
@@
 	1    0    0    -1
 $EndComp
-Wire Wire Line
-	9100 2550 9500 2550
 Connection ~ 9500 2250
-Wire Wire Line
-	9500 2250 9500 2550
-Connection ~ 9500 2550
-Text GLabel 1250 2550 0    50   Input ~ 0
-row1
 Wire Wire Line
 	1250 2550 1400 2550
@@
 Wire Wire Line
 	8950 1800 8950 2250
-Wire Wire Line
-	9500 1800 9500 2250
 $Comp
 L Device:D D31
@@
 	1    0    0    -1
 $EndComp
-Wire Wire Line
-	9100 3300 9500 3300
 Connection ~ 9500 3000
-Wire Wire Line
-	9500 3000 9500 3300
-Connection ~ 9500 3300
-Text GLabel 1250 3300 0    50   Input ~ 0
-row2
 Wire Wire Line
 	1250 3300 1400 3300
@@
 	1    0    0    -1
 $EndComp
-Wire Wire Line
-	9100 4050 9500 4050
 Connection ~ 9500 3750
-Wire Wire Line
-	9500 3750 9500 4050
-Connection ~ 9500 4050
-Text GLabel 1250 4050 0    50   Input ~ 0
-row3
 Wire Wire Line
 	1250 4050 1400 4050
@@
 	8950 3300 8950 3750
 Wire Wire Line
-	9500 3300 9500 3750
-Wire Wire Line
 	1800 2550 1800 3000
 Wire Wire Line
@@
 Wire Wire Line
 	8950 2550 8950 3000
-Wire Wire Line
-	9500 2550 9500 3000
 $Comp
 L Device:D D59
@@
 	1    0    0    -1
 $EndComp
-Text GLabel 1250 4800 0    50   Input ~ 0
-row4
 Wire Wire Line
 	1250 4800 1400 4800
@@
 Wire Wire Line
 	8950 4050 8950 4500
-Wire Wire Line
-	9500 4050 9500 4500
+Connection ~ 7850 4800
+Wire Wire Line
+	7850 4050 7850 4500
+Wire Wire Line
+	7850 4500 7850 4800
+Connection ~ 7850 4500
+Wire Wire Line
+	7300 4050 7300 4500
+Wire Wire Line
+	7450 4800 7850 4800
+$Comp
+L Switch:SW_Push SW64
+U 1 1 64854FF7
+P 7650 4500
+F 0 "SW64" H 7650 4785 50  0000 C CNN
+F 1 "0" H 7650 4694 50  0000 C CNN
+F 2 "Alps_Only:ALPS-1U" H 7650 4700 50  0001 C CNN
+F 3 "~" H 7650 4700 50  0001 C CNN
+	1    7650 4500
+	1    0    0    -1
+$EndComp
+$Comp
+L Device:D D64
+U 1 1 64854FF1
+P 7450 4650
+F 0 "D64" V 7496 4571 50  0000 R CNN
+F 1 "D" V 7405 4571 50  0000 R CNN
+F 2 "Diode_SMD:D_SOD-123" H 7450 4650 50  0001 C CNN
+F 3 "~" H 7450 4650 50  0001 C CNN
+	1    7450 4650
+	0    -1   -1   0
+$EndComp
+Wire Wire Line
+	7450 4800 7300 4800
+Connection ~ 7300 4800
+Wire Wire Line
+	7300 4500 7300 4800
+Connection ~ 7300 4500
+Wire Wire Line
+	6900 4800 7300 4800
+$Comp
+L Switch:SW_Push SW63
+U 1 1 64854FE5
+P 7100 4500
+F 0 "SW63" H 7100 4785 50  0000 C CNN
+F 1 "ralt" H 7100 4694 50  0000 C CNN
+F 2 "Alps_Only:ALPS-1.25U" H 7100 4700 50  0001 C CNN
+F 3 "~" H 7100 4700 50  0001 C CNN
+	1    7100 4500
+	1    0    0    -1
+$EndComp
+$Comp
+L Device:D D63
+U 1 1 64854FDF
+P 6900 4650
+F 0 "D63" V 6946 4571 50  0000 R CNN
+F 1 "D" V 6855 4571 50  0000 R CNN
+F 2 "Diode_SMD:D_SOD-123" H 6900 4650 50  0001 C CNN
+F 3 "~" H 6900 4650 50  0001 C CNN
+	1    6900 4650
+	0    -1   -1   0
+$EndComp
+$Comp
+L Device:D D62
+U 1 1 648EC32B
+P 4700 4650
+F 0 "D62" V 4746 4571 50  0000 R CNN
+F 1 "D" V 4655 4571 50  0000 R CNN
+F 2 "Diode_SMD:D_SOD-123" H 4700 4650 50  0001 C CNN
+F 3 "~" H 4700 4650 50  0001 C CNN
+	1    4700 4650
+	0    -1   -1   0
+$EndComp
+$Comp
+L Switch:SW_Push SW62
+U 1 1 648EC331
+P 4900 4500
+F 0 "SW62" H 4900 4785 50  0000 C CNN
+F 1 "spacebar" H 4900 4694 50  0000 C CNN
+F 2 "Alps_Only:ALPS-6.5U" H 4900 4700 50  0001 C CNN
+F 3 "~" H 4900 4700 50  0001 C CNN
+	1    4900 4500
+	1    0    0    -1
+$EndComp
+Wire Wire Line
+	5100 4050 5100 4500
+Wire Wire Line
+	2500 4800 4700 4800
+Wire Wire Line
+	4700 4800 6900 4800
+Wire Wire Line
+	7850 3300 7850 4050
+Connection ~ 7300 3750
+Wire Wire Line
+	7300 3750 7300 4050
+Wire Wire Line
+	8400 2550 8400 3300
+Wire Wire Line
+	7850 3300 8400 3300
+Wire Wire Line
+	7300 4050 7850 4050
 Text GLabel 1800 1200 1    50   Input ~ 0
 col0
+Wire Wire Line
+	9500 3750 9500 4500
+Wire Wire Line
+	9500 3000 9500 3750
+Wire Wire Line
+	9500 2250 9500 3000
+Wire Wire Line
+	9500 1500 9500 2250
 Text GLabel 2350 1200 1    50   Input ~ 0
 col1
@@
 Text GLabel 9500 1200 1    50   Input ~ 0
 col14
-Connection ~ 7850 4800
-Wire Wire Line
-	7850 4050 7850 4500
-Wire Wire Line
-	7850 4500 7850 4800
-Connection ~ 7850 4500
-Wire Wire Line
-	7300 4050 7300 4500
-Wire Wire Line
-	7450 4800 7850 4800
-$Comp
-L Switch:SW_Push SW64
-U 1 1 64854FF7
-P 7650 4500
-F 0 "SW64" H 7650 4785 50  0000 C CNN
-F 1 "0" H 7650 4694 50  0000 C CNN
-F 2 "Alps_Only:ALPS-1U" H 7650 4700 50  0001 C CNN
-F 3 "~" H 7650 4700 50  0001 C CNN
-	1    7650 4500
-	1    0    0    -1
-$EndComp
-$Comp
-L Device:D D64
-U 1 1 64854FF1
-P 7450 4650
-F 0 "D64" V 7496 4571 50  0000 R CNN
-F 1 "D" V 7405 4571 50  0000 R CNN
-F 2 "Diode_SMD:D_SOD-123" H 7450 4650 50  0001 C CNN
-F 3 "~" H 7450 4650 50  0001 C CNN
-	1    7450 4650
-	0    -1   -1   0
-$EndComp
-Wire Wire Line
-	7450 4800 7300 4800
-Connection ~ 7300 4800
-Wire Wire Line
-	7300 4500 7300 4800
-Connection ~ 7300 4500
-Wire Wire Line
-	6900 4800 7300 4800
-$Comp
-L Switch:SW_Push SW63
-U 1 1 64854FE5
-P 7100 4500
-F 0 "SW63" H 7100 4785 50  0000 C CNN
-F 1 "ralt" H 7100 4694 50  0000 C CNN
-F 2 "Alps_Only:ALPS-1.25U" H 7100 4700 50  0001 C CNN
-F 3 "~" H 7100 4700 50  0001 C CNN
-	1    7100 4500
-	1    0    0    -1
-$EndComp
-$Comp
-L Device:D D63
-U 1 1 64854FDF
-P 6900 4650
-F 0 "D63" V 6946 4571 50  0000 R CNN
-F 1 "D" V 6855 4571 50  0000 R CNN
-F 2 "Diode_SMD:D_SOD-123" H 6900 4650 50  0001 C CNN
-F 3 "~" H 6900 4650 50  0001 C CNN
-	1    6900 4650
-	0    -1   -1   0
-$EndComp
-$Comp
-L Device:D D62
-U 1 1 648EC32B
-P 4700 4650
-F 0 "D62" V 4746 4571 50  0000 R CNN
-F 1 "D" V 4655 4571 50  0000 R CNN
-F 2 "Diode_SMD:D_SOD-123" H 4700 4650 50  0001 C CNN
-F 3 "~" H 4700 4650 50  0001 C CNN
-	1    4700 4650
-	0    -1   -1   0
-$EndComp
-$Comp
-L Switch:SW_Push SW62
-U 1 1 648EC331
-P 4900 4500
-F 0 "SW62" H 4900 4785 50  0000 C CNN
-F 1 "spacebar" H 4900 4694 50  0000 C CNN
-F 2 "Alps_Only:ALPS-6.5U" H 4900 4700 50  0001 C CNN
-F 3 "~" H 4900 4700 50  0001 C CNN
-	1    4900 4500
-	1    0    0    -1
-$EndComp
-Wire Wire Line
-	5100 4050 5100 4500
-Wire Wire Line
-	2500 4800 4700 4800
-Wire Wire Line
-	4700 4800 6900 4800
-Wire Wire Line
-	7850 3300 7850 4050
-Connection ~ 7300 3750
-Wire Wire Line
-	7300 3750 7300 4050
-Wire Wire Line
-	8400 2550 8400 3300
-Wire Wire Line
-	7850 3300 8400 3300
-Wire Wire Line
-	7300 4050 7850 4050
+Text GLabel 1250 1800 0    50   Input ~ 0
+row0
+Text GLabel 1250 2550 0    50   Input ~ 0
+row1
+Text GLabel 1250 3300 0    50   Input ~ 0
+row2
+Text GLabel 1250 4050 0    50   Input ~ 0
+row3
+Text GLabel 1250 4800 0    50   Input ~ 0
+row4
 $EndSCHEMATC
